File: Documentation/Wiring_Diagram/Avera_G60_Wiring_Diagram.kicad_sch (KiCad schematic)
At the start: 15 parts

Commit message: create png logo
Parts:
- 100K_LINEAR: value (none) -> SLIDER POT DUAL GANG - PICKUP BLEND
- 500K_AUDIO: value (none) -> PUSH PULL POT - TONE
- 500K_AUDIO: value (none) -> PUSH PULL POT - VOLUME
- C?: value (none) -> C
- RV?: value (none) -> PICKUP BLEND
Changed lines of the file:
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@@
   )
   (wire (pts (xy 127 133.35) (xy 127 96.52))
-    (stroke (width 0) (type default) (color 255 153 0 1))
+    (stroke (width 0) (type default) (color 255 255 0 1))
   )
   (wire (pts (xy 181.61 91.44) (xy 181.61 97.79))
@@
   )
   (wire (pts (xy 72.39 133.35) (xy 72.39 83.82))
-    (stroke (width 0) (type default) (color 255 153 0 1))
+    (stroke (width 0) (type default) (color 255 255 0 1))
   )
   (polyline (pts (xy 161.29 92.71) (xy 179.07 92.71))
@@
   )
   (wire (pts (xy 78.74 133.35) (xy 72.39 133.35))
-    (stroke (width 0) (type default) (color 255 153 0 1))
+    (stroke (width 0) (type default) (color 255 255 0 1))
   )
   (polyline (pts (xy 179.07 92.71) (xy 179.07 85.09))
@@
   )
   (wire (pts (xy 72.39 83.82) (xy 127 83.82))
-    (stroke (width 0) (type default) (color 255 153 0 1))
+    (stroke (width 0) (type default) (color 255 255 0 1))
   )
   (wire (pts (xy 158.75 128.27) (xy 158.75 111.76))
@@
   )
   (wire (pts (xy 101.6 133.35) (xy 127 133.35))
-    (stroke (width 0) (type default) (color 255 153 0 1))
+    (stroke (width 0) (type default) (color 255 255 0 1))
   )
   (wire (pts (xy 101.6 81.28) (xy 69.85 81.28))
@@
   )
   (wire (pts (xy 127 83.82) (xy 127 85.09))
-    (stroke (width 0) (type default) (color 255 153 0 1))
+    (stroke (width 0) (type default) (color 255 255 0 1))
   )
   (wire (pts (xy 156.21 138.43) (xy 168.91 138.43))
@@
       (effects (font (size 1.27 1.27)) hide)
     )
-    (property "Value" "" (id 1) (at 100.33 124.46 0)
+    (property "Value" "Earth" (id 1) (at 100.33 124.46 0)
       (effects (font (size 1.27 1.27)) hide)
     )
@@
     (in_bom yes) (on_board yes)
     (property "Reference" "100K_LINEAR" (id 0) (at 127 81.28 90))
-    (property "Value" "" (id 1) (at 127 78.74 90))
+    (property "Value" "SLIDER POT DUAL GANG - PICKUP BLEND" (id 1) (at 127 78.74 90))
     (property "Footprint" "" (id 2) (at 127 88.9 0)
       (effects (font (size 1.27 1.27)) hide)
@@
     (in_bom yes) (on_board yes)
     (property "Reference" "500K_AUDIO" (id 0) (at 170.18 118.11 90))
-    (property "Value" "" (id 1) (at 170.18 115.57 90))
+    (property "Value" "PUSH PULL POT - TONE" (id 1) (at 170.18 115.57 90))
     (property "Footprint" "" (id 2) (at 170.18 124.46 0)
       (effects (font (size 1.27 1.27)) hide)
@@
       (effects (font (size 1.27 1.27)) (justify left))
     )
-    (property "Value" "" (id 1) (at 168.91 105.41 0)
+    (property "Value" "C" (id 1) (at 168.91 105.41 0)
       (effects (font (size 1.27 1.27)) (justify left))
     )
@@
       (effects (font (size 1.27 1.27)) hide)
     )
-    (property "Value" "" (id 1) (at 119.38 97.79 90)
+    (property "Value" "PICKUP BLEND" (id 1) (at 119.38 97.79 90)
       (effects (font (size 1.27 1.27)) hide)
     )
@@
     (in_bom yes) (on_board yes)
     (property "Reference" "500K_AUDIO" (id 0) (at 91.44 116.84 90))
-    (property "Value" "" (id 1) (at 92.71 114.3 90))
+    (property "Value" "PUSH PULL POT - VOLUME" (id 1) (at 92.71 114.3 90))
     (property "Footprint" "" (id 2) (at 90.17 124.46 0)
       (effects (font (size 1.27 1.27)) hide)

Commit message: update CAM files and make wiring diagram pdf
Parts:
- C0.0022: renamed from C?; value C -> (none)
- C?: value C -> (none)
- J?: value Jack-DC -> (none)
- gave numbers to parts that had none: 1
- renumbered 500K_AUDIO to 500K_LOG
Other:
- note removed: "PHASE SWITCH"
