File: Documentation/Wiring_Diagram/Avera_G60_Wiring_Diagram_Light.kicad_sch (KiCad schematic)
At the start: 15 parts

Commit message: update wiring diagram
Other:
- company: (none) -> Orion Miller
- title: (none) -> Avera G-60 Wiring Diagram
Changed lines of the file:
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@@
 (kicad_sch (version 20211123) (generator eeschema)
   (paper "A4")
-  (junction (at 158.75 97.79) (diameter 0) (color 255 153 0 1)
+  (title_block
+    (title "Avera G-60 Wiring Diagram")
+    (date "2024-01-17")
+    (company "Orion Miller")
+  )
+  (junction (at 158.75 97.79) (diameter 0) (color 255 255 0 1)
   )
   (junction (at 181.61 91.44) (diameter 0) (color 255 255 255 1)
@@
   (junction (at 168.91 130.81) (diameter 0) (color 0 0 0 0)
   )
-  (junction (at 123.19 92.71) (diameter 0) (color 255 0 255 1)
+  (junction (at 123.19 92.71) (diameter 0) (color 90 153 255 1)
   )
   (junction (at 101.6 83.82) (diameter 0) (color 255 153 0 1)
@@
   (junction (at 158.75 147.32) (diameter 0) (color 255 0 0 1)
   )
-  (junction (at 153.67 97.79) (diameter 0) (color 255 153 0 1)
+  (junction (at 153.67 97.79) (diameter 0) (color 255 255 0 1)
   )
   (wire (pts (xy 181.61 91.44) (xy 181.61 95.25))
@@
   )
   (wire (pts (xy 123.19 90.17) (xy 123.19 92.71))
-    (stroke (width 0) (type default) (color 255 0 255 1))
+    (stroke (width 0) (type default) (color 90 153 255 1))
   )
   (polyline (pts (xy 93.98 120.65) (xy 93.98 127))
@@
   )
   (wire (pts (xy 90.17 120.65) (xy 90.17 119.38))
-    (stroke (width 0) (type default) (color 255 0 255 1))
+    (stroke (width 0) (type default) (color 90 153 255 1))
   )
   (polyline (pts (xy 179.07 85.09) (xy 161.29 85.09))
@@
   )
   (wire (pts (xy 88.9 130.81) (xy 88.9 129.54))
-    (stroke (width 0) (type default) (color 255 0 255 1))
+    (stroke (width 0) (type default) (color 90 153 255 1))
   )
   (wire (pts (xy 76.2 133.35) (xy 78.74 133.35))
-    (stroke (width 0) (type default) (color 255 0 255 1))
+    (stroke (width 0) (type default) (color 90 153 255 1))
   )
   (wire (pts (xy 85.09 129.54) (xy 85.09 124.46))
-    (stroke (width 0) (type default) (color 255 0 255 1))
+    (stroke (width 0) (type default) (color 90 153 255 1))
   )
   (polyline (pts (xy 166.37 120.65) (xy 173.99 120.65))
@@
   )
   (wire (pts (xy 85.09 124.46) (xy 86.36 124.46))
-    (stroke (width 0) (type default) (color 255 0 255 1))
+    (stroke (width 0) (type default) (color 90 153 255 1))
   )
   (wire (pts (xy 130.81 90.17) (xy 123.19 90.17))
-    (stroke (width 0) (type default) (color 255 0 255 1))
+    (stroke (width 0) (type default) (color 90 153 255 1))
   )
   (wire (pts (xy 73.66 137.16) (xy 91.44 137.16))
@@
   )
   (wire (pts (xy 127 83.82) (xy 127 85.09))
-    (stroke (width 0) (type default) (color 255 153 0 1))
+    (stroke (width 0) (type default) (color 255 255 0 1))
   )
   (wire (pts (xy 156.21 137.16) (xy 168.91 137.16))
-    (stroke (width 0) (type default) (color 255 0 255 1))
+    (stroke (width 0) (type default) (color 90 153 255 1))
   )
   (wire (pts (xy 130.81 92.71) (xy 133.35 92.71))
@@
   )
   (wire (pts (xy 90.17 119.38) (xy 156.21 119.38))
-    (stroke (width 0) (type default) (color 255 0 255 1))
+    (stroke (width 0) (type default) (color 90 153 255 1))
   )
   (wire (pts (xy 134.62 147.32) (xy 158.75 147.32))
@@
   )
   (wire (pts (xy 130.81 88.9) (xy 130.81 90.17))
-    (stroke (width 0) (type default) (color 255 0 255 1))
+    (stroke (width 0) (type default) (color 90 153 255 1))
   )
   (wire (pts (xy 78.74 83.82) (xy 101.6 83.82))
-    (stroke (width 0) (type default) (color 255 153 0 1))
+    (stroke (width 0) (type default) (color 255 255 0 1))
   )
   (wire (pts (xy 181.61 91.44) (xy 186.69 91.44))
@@
   )
   (wire (pts (xy 127 96.52) (xy 127 97.79))
-    (stroke (width 0) (type default) (color 255 153 0 1))
-  )
-  (polyline (pts (xy 130.81 96.52) (xy 130.81 85.09))
-    (stroke (width 0) (type default) (color 0 132 132 1))
+    (stroke (width 0) (type default) (color 255 255 0 1))
   )
   (polyline (pts (xy 86.36 120.65) (xy 93.98 120.65))
@@
   )
   (wire (pts (xy 156.21 119.38) (xy 156.21 137.16))
-    (stroke (width 0) (type default) (color 255 0 255 1))
+    (stroke (width 0) (type default) (color 90 153 255 1))
   )
   (wire (pts (xy 168.91 34.29) (xy 168.91 38.1))
@@
   )
   (wire (pts (xy 153.67 97.79) (xy 158.75 97.79))
-    (stroke (width 0) (type default) (color 255 153 0 1))
+    (stroke (width 0) (type default) (color 255 255 0 1))
   )
   (wire (pts (xy 86.36 34.29) (xy 101.6 34.29))
@@
   )
   (wire (pts (xy 76.2 92.71) (xy 123.19 92.71))
-    (stroke (width 0) (type default) (color 255 0 255 1))
+    (stroke (width 0) (type default) (color 90 153 255 1))
   )
   (polyline (pts (xy 123.19 85.09) (xy 123.19 96.52))
@@
   )
   (wire (pts (xy 78.74 83.82) (xy 78.74 128.27))
-    (stroke (width 0) (type default) (color 255 153 0 1))
+    (stroke (width 0) (type default) (color 255 255 0 1))
   )
   (wire (pts (xy 184.15 86.36) (xy 184.15 97.79))
-    (stroke (width 0) (type default) (color 255 153 0 1))
+    (stroke (width 0) (type default) (color 255 255 0 1))
   )
   (polyline (pts (xy 99.06 134.62) (xy 99.06 127))
@@
   )
   (wire (pts (xy 76.2 92.71) (xy 76.2 133.35))
-    (stroke (width 0) (type default) (color 255 0 255 1))
+    (stroke (width 0) (type default) (color 90 153 255 1))
   )
   (wire (pts (xy 168.91 137.16) (xy 168.91 130.81))
-    (stroke (width 0) (type default) (color 255 0 255 1))
+    (stroke (width 0) (type default) (color 90 153 255 1))
+  )
+  (polyline (pts (xy 130.81 85.09) (xy 130.81 96.52))
+    (stroke (width 0) (type default) (color 0 132 132 1))
   )
   (wire (pts (xy 168.91 63.5) (xy 168.91 88.9))
@@
   )
   (wire (pts (xy 88.9 129.54) (xy 85.09 129.54))
-    (stroke (width 0) (type default) (color 255 0 255 1))
+    (stroke (width 0) (type default) (color 90 153 255 1))
   )
   (wire (pts (xy 158.75 91.44) (xy 158.75 97.79))
-    (stroke (width 0) (type default) (color 255 153 0 1))
+    (stroke (width 0) (type default) (color 255 255 0 1))
   )
   (polyline (pts (xy 81.28 134.62) (xy 99.06 134.62))
@@
   )
   (wire (pts (xy 153.67 97.79) (xy 153.67 128.27))
-    (stroke (width 0) (type default) (color 255 153 0 1))
+    (stroke (width 0) (type default) (color 255 255 0 1))
   )
   (wire (pts (xy 86.36 66.04) (xy 73.66 66.04))
@@
   )
   (wire (pts (xy 181.61 86.36) (xy 184.15 86.36))
-    (stroke (width 0) (type default) (color 255 153 0 1))
+    (stroke (width 0) (type default) (color 255 255 0 1))
   )
   (wire (pts (xy 153.67 128.27) (xy 101.6 128.27))
-    (stroke (width 0) (type default) (color 255 153 0 1))
+    (stroke (width 0) (type default) (color 255 255 0 1))
   )
   (wire (pts (xy 181.61 133.35) (xy 184.15 133.35))
@@
   )
   (wire (pts (xy 101.6 83.82) (xy 127 83.82))
-    (stroke (width 0) (type default) (color 255 153 0 1))
+    (stroke (width 0) (type default) (color 255 255 0 1))
   )
   (wire (pts (xy 158.75 97.79) (xy 184.15 97.79))
-    (stroke (width 0) (type default) (color 255 153 0 1))
+    (stroke (width 0) (type default) (color 255 255 0 1))
   )
   (wire (pts (xy 127 97.79) (xy 153.67 97.79))
-    (stroke (width 0) (type default) (color 255 153 0 1))
+    (stroke (width 0) (type default) (color 255 255 0 1))
   )
   (wire (pts (xy 171.45 128.27) (xy 171.45 130.81))
